File: current/new current sensor.kicad_pcb (KiCad board)
At the start: 2 copper layers, 151.3 x 62.3 mm, 51 parts, among them J1 Conn_01x04, U1 ACS711xEXLT-31AB, U2 ACS711xEXLT-31AB, U3 ACS711xEXLT-31AB, U4 ACS711xEXLT-31AB, U5 ACS711xEXLT-31AB, U6 ACS711xEXLT-31AB, U7 ADS1119IPWR, U8 ADS1119IPWR

Commit message: final tweaks before ordering
Parts:
- added REF**: MountingHole_3.7mm_Pad, MountingHole:MountingHole_3.7mm_Pad, F.Cu at (241.3, 38.1)
- added REF**: MountingHole_3.7mm_Pad, MountingHole:MountingHole_3.7mm_Pad, F.Cu at (108.0, 82.5)
- added REF**: MountingHole_3.7mm_Pad, MountingHole:MountingHole_3.7mm_Pad, F.Cu at (108.0, 38.1)
- added REF**: MountingHole_3.7mm_Pad, MountingHole:MountingHole_3.7mm_Pad, F.Cu at (241.3, 82.5)
Connections:
- J1 pad 3: +3.3V -> +3V3
Routing:
- net +3.3V: track 239.7 -> 238.9 mm
- net Net-(U5-VIOUT): track 28.3 -> 27.7 mm
Other:
- board size 151.3 x 62.3 mm -> 151.3 x 57 mm
