File: new current sensor.kicad_pcb (KiCad board)
At the start: 2 copper layers, 151.3 x 62.3 mm, 57 parts, among them J1 Conn_01x04, U1 ACS711xEXLT-31AB, U2 ACS711xEXLT-31AB, U3 ACS711xEXLT-31AB, U4 ACS711xEXLT-31AB, U5 ACS711xEXLT-31AB, U6 ACS711xEXLT-31AB, U7 ADS1119IPWR, U8 ADS1119IPWR

Commit message: final changes
Routing:
- net Net-(J1-Pad2): track 40.7 -> 42.2 mm
Changed lines of the file:
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@@
   (segment (start 211.0525 57.975) (end 212.095 57.975) (width 0.25) (layer "F.Cu") (net 2))
   (segment (start 206.1 67.2) (end 205.8 66.9) (width 0.25) (layer "F.Cu") (net 2))
+  (segment (start 138.1375 59.6375) (end 138.1375 56.422203) (width 0.25) (layer "F.Cu") (net 2))
   (segment (start 228.2334 55.6232) (end 228.2334 53.848) (width 0.25) (layer "F.Cu") (net 2))
   (segment (start 167.35 55.2) (end 167.1 55.2) (width 0.25) (layer "F.Cu") (net 2))
@@
   (segment (start 226.9352 53.848) (end 226.9352 54.9114) (width 0.25) (layer "F.Cu") (net 2))
   (segment (start 226.6798 65.725) (end 226.6298 65.775) (width 0.25) (layer "F.Cu") (net 2))
-  (segment (start 138.4 59.65) (end 138.1375 59.3875) (width 0.25) (layer "F.Cu") (net 2))
   (segment (start 202.1 54.6) (end 202.85 54.6) (width 0.25) (layer "F.Cu") (net 2))
   (segment (start 230.9368 76.1492) (end 230.9368 77.8117) (width 0.25) (layer "F.Cu") (net 2))
@@
   (segment (start 130.890395 54.980395) (end 131.114895 55.204895) (width 0.25) (layer "F.Cu") (net 2))
   (segment (start 198.325 63.995) (end 198.325 65.9) (width 0.25) (layer "F.Cu") (net 2))
+  (segment (start 138.5 60) (end 138.1375 59.6375) (width 0.25) (layer "F.Cu") (net 2))
   (segment (start 210.825 56.07) (end 210.825 57.7475) (width 0.25) (layer "F.Cu") (net 2))
   (segment (start 226.9352 54.9114) (end 226.2742 55.5724) (width 0.25) (layer "F.Cu") (net 2))
   (segment (start 229.2298 64.55) (end 229.2298 65.775) (width 0.25) (layer "F.Cu") (net 2))
-  (segment (start 138.1375 59.3875) (end 138.1375 56.422203) (width 0.25) (layer "F.Cu") (net 2))
   (segment (start 228.8368 76.1117) (end 228.8368 77.8017) (width 0.25) (layer "F.Cu") (net 2))
   (segment (start 228.8834 54.9732) (end 228.8834 53.848) (width 0.25) (layer "F.Cu") (net 2))
@@
   (via (at 228.8368 77.8017) (size 0.8) (drill 0.4) (layers "F.Cu" "B.Cu") (free) (net 2))
   (via (at 224.8916 40.132) (size 0.8) (drill 0.4) (layers "F.Cu" "B.Cu") (net 2))
-  (via (at 138.4 59.65) (size 0.8) (drill 0.4) (layers "F.Cu" "B.Cu") (net 2))
+  (via (at 138.5 60) (size 0.8) (drill 0.4) (layers "F.Cu" "B.Cu") (net 2))
   (via (at 134.5 67.5) (size 0.8) (drill 0.4) (layers "F.Cu" "B.Cu") (net 2))
   (via (at 228.5798 63.9) (size 0.8) (drill 0.4) (layers "F.Cu" "B.Cu") (net 2))
@@
   (segment (start 236.8872 62.1192) (end 243.8444 62.1192) (width 0.25) (layer "F.Cu") (net 37))
   (segment (start 234.2388 64.8716) (end 234.2388 59.9092) (width 0.25) (layer "F.Cu") (net 37))
+  (segment (start 230.324 51) (end 234.2388 54.9148) (width 0.25) (layer "F.Cu") (net 37))
+  (segment (start 226.9352 48.810861) (end 229.124339 51) (width 0.25) (layer "F.Cu") (net 37))
   (segment (start 234.2388 59.9092) (end 234.458 59.69) (width 0.25) (layer "F.Cu") (net 37))
-  (segment (start 232.0544 69.287539) (end 232.0544 68.5292) (width 0.25) (layer "F.Cu") (net 37))
   (segment (start 234.458 59.69) (end 236.8872 62.1192) (width 0.25) (layer "F.Cu") (net 37))
   (segment (start 234.2388 54.9148) (end 234.2388 59.3504) (width 0.25) (layer "F.Cu") (net 37))
-  (segment (start 230.5298 70.812139) (end 232.0544 69.287539) (width 0.25) (layer "F.Cu") (net 37))
+  (segment (start 230.5298 70.0538) (end 232.0544 68.5292) (width 0.25) (layer "F.Cu") (net 37))
+  (segment (start 229.124339 51) (end 230.324 51) (width 0.25) (layer "F.Cu") (net 37))
+  (segment (start 230.5298 71.5) (end 230.5298 70.0538) (width 0.25) (layer "F.Cu") (net 37))
   (segment (start 226.9352 48.123) (end 226.9352 48.810861) (width 0.25) (layer "F.Cu") (net 37))
-  (segment (start 227.309359 49.18502) (end 228.50902 49.18502) (width 0.25) (layer "F.Cu") (net 37))
-  (segment (start 228.50902 49.18502) (end 234.2388 54.9148) (width 0.25) (layer "F.Cu") (net 37))
-  (segment (start 230.5298 71.5) (end 230.5298 70.812139) (width 0.25) (layer "F.Cu") (net 37))
-  (segment (start 226.9352 48.810861) (end 227.309359 49.18502) (width 0.25) (layer "F.Cu") (net 37))
   (via (at 232.0544 68.5292) (size 0.8) (drill 0.4) (layers "F.Cu" "B.Cu") (net 37))
   (via (at 234.2388 64.8716) (size 0.8) (drill 0.4) (layers "F.Cu" "B.Cu") (net 37))
   (segment (start 234.2388 66.3448) (end 234.2388 64.8716) (width 0.25) (layer "B.Cu") (net 37))
   (segment (start 232.0544 68.5292) (end 234.2388 66.3448) (width 0.25) (layer "B.Cu") (net 37))
-  (segment (start 226.2852 48.810861) (end 227.108879 49.63454) (width 0.25) (layer "F.Cu") (net 38))
-  (segment (start 226.2852 48.123) (end 226.2852 48.810861) (width 0.25) (layer "F.Cu") (net 38))
+  (segment (start 228.987169 52) (end 226.2852 49.298031) (width 0.25) (layer "F.Cu") (net 38))
   (segment (start 232.9688 61.2808) (end 231.378 59.69) (width 0.25) (layer "F.Cu") (net 38))
-  (segment (start 227.959601 49.63454) (end 233.2736 54.948539) (width 0.25) (layer "F.Cu") (net 38))
+  (segment (start 233.1396 54.814539) (end 233.1396 57.9284) (width 0.25) (layer "F.Cu") (net 38))
   (segment (start 232.9688 69.711) (end 232.9688 61.2808) (width 0.25) (layer "F.Cu") (net 38))
-  (segment (start 233.2736 57.4548) (end 233.2736 57.5056) (width 0.25) (layer "F.Cu") (net 38))
+  (segment (start 233.1396 54.814539) (end 230.325061 52) (width 0.25) (layer "F.Cu") (net 38))
+  (segment (start 230.325061 52) (end 228.987169 52) (width 0.25) (layer "F.Cu") (net 38))
   (segment (start 231.1798 71.5) (end 232.9688 69.711) (width 0.25) (layer "F.Cu") (net 38))
-  (segment (start 233.2736 57.5056) (end 231.4448 59.3344) (width 0.25) (layer "F.Cu") (net 38))
-  (segment (start 227.108879 49.63454) (end 227.959601 49.63454) (width 0.25) (layer "F.Cu") (net 38))
+  (segment (start 232.81 59.69) (end 231.378 59.69) (width 0.25) (layer "F.Cu") (net 38))
   (segment (start 243.4072 59.182) (end 243.8444 59.6192) (width 0.25) (layer "F.Cu") (net 38))
-  (segment (start 233.2736 54.948539) (end 233.2736 57.4548) (width 0.25) (layer "F.Cu") (net 38))
-  (via (at 233.2736 57.4548) (size 0.8) (drill 0.4) (layers "F.Cu" "B.Cu") (net 38))
-  (segment (start 240.6192 59.6192) (end 243.8444 59.6192) (width 0.25) (layer "B.Cu") (net 38))
-  (segment (start 238.4548 57.4548) (end 240.6192 59.6192) (width 0.25) (layer "B.Cu") (net 38))
-  (segment (start 233.2736 57.4548) (end 238.4548 57.4548) (width 0.25) (layer "B.Cu") (net 38))
+  (segment (start 226.2852 49.298031) (end 226.2852 48.123) (width 0.25) (layer "F.Cu") (net 38))
+  (segment (start 233.1396 57.9284) (end 231.378 59.69) (width 0.25) (layer "F.Cu") (net 38))
+  (via (at 232.81 59.69) (size 0.5) (drill 0.3) (layers "F.Cu" "B.Cu") (net 38))
+  (segment (start 243.8444 59.6192) (end 232.8808 59.6192) (width 0.25) (layer "B.Cu") (net 38))
+  (segment (start 232.8808 59.6192) (end 232.81 59.69) (width 0.25) (layer "B.Cu") (net 38))
   (segment (start 230.6 45.89) (end 230.6 46.45) (width 0.25) (layer "F.Cu") (net 43))
   (segment (start 230.6 46.45) (end 230.1852 46.8648) (width 0.25) (layer "F.Cu") (net 43))

Commit message: added tps
Parts:
- added TP10: 3.3V, Connector_Wire:SolderWire-0.1sqmm_1x01_D0.4mm_OD1mm, F.Cu at (240.0, 44.5)
- added TP7: SCL, Connector_Wire:SolderWire-0.1sqmm_1x01_D0.4mm_OD1mm, F.Cu at (244.0, 75.0)
- added TP8: SDA, Connector_Wire:SolderWire-0.1sqmm_1x01_D0.4mm_OD1mm, F.Cu at (244.0, 69.0)
- added TP9: GND, Connector_Wire:SolderWire-0.1sqmm_1x01_D0.4mm_OD1mm, F.Cu at (240.0, 49.0)
Connections:
- net Net-(J1-Pad1) renamed /SDA
- net Net-(J1-Pad2) renamed /SCL
Routing:
- net /SCL: track 42.2 -> 61.4 mm
- net /SDA: track 38.8 -> 45.7 mm
Other:
- board text added: "+3.3V"
- board text added: "Actuation Left"
- board text added: "Actuation Right"
- board text added: "Deposition"
- board text added: "Drive Left"
- board text added: "Drive Right"
- board text added: "Excavation"
- board text removed: "+3V3"

Commit message: done now
Routing:
- net Net-(U4-~{FAULT}): track 5.93 -> 4.36 mm
Changed lines of the file:
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@@
   (segment (start 172.6 64.7) (end 175.6 64.7) (width 0.25) (layer "F.Cu") (net 16))
   (segment (start 169.5 66.45) (end 170.85 66.45) (width 0.25) (layer "F.Cu") (net 16))
+  (segment (start 165.4325 55.7) (end 165.3975 55.665) (width 0.25) (layer "F.Cu") (net 17))
   (segment (start 164.995 55.665) (end 164.995 57.57) (width 0.25) (layer "F.Cu") (net 17))
-  (segment (start 164.845 58.205) (end 167.35 55.7) (width 0.25) (layer "F.Cu") (net 17))
+  (segment (start 167.35 55.7) (end 165.4325 55.7) (width 0.25) (layer "F.Cu") (net 17))
   (segment (start 164.36 58.205) (end 164.845 58.205) (width 0.25) (layer "F.Cu") (net 17))
   (segment (start 201.38 55.75) (end 200.965 56.165) (width 0.25) (layer "F.Cu") (net 18))
